Commit message: Update pioneer3at.urdf

File: src/p3at_qlearning_simulation_v2/urdf/pioneer3at.urdf (robot description, URDF)
Before this commit: robot pioneer3at, 20 links, 19 joints
Links:
- removed link back_sonar
- removed link cam_link
- removed link front_sonar
- removed link p3at_back_left_axle
- removed link p3at_back_left_hub
- removed link p3at_back_left_wheel
- removed link p3at_back_right_axle
- removed link p3at_back_right_hub
- removed link p3at_back_right_wheel
- removed link p3at_front_left_axle
- removed link p3at_front_left_hub
- removed link p3at_front_left_wheel
- removed link p3at_front_right_axle
- removed link p3at_front_right_hub
- removed link p3at_front_right_wheel
- removed link pantbl_link
- link base_cam: mass 1e-5 -> None; geometry visual cylinder length=0.01 radius=0.02
- link base_link: geometry collision mesh filename=package://p3at_qlearning_simulation_v2/meshes/p3at_meshes/c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; visual mesh filename=package://p3at_qlearning_simulation_v2/meshes/p3at_meshes/c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
- link hokuyo: mass 1e-5 -> None; geometry visual mesh filename=package://p3at_qlearning_simulation_v2/meshes/hokuyo.dae
- link top_plate: geometry visual mesh filename=package://p3at_qlearning_simulation_v2/meshes/p3at_meshes/t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
Joints:
- removed joint base_back_joint
- removed joint base_front_joint
- removed joint base_front_left_axle_joint
- removed joint base_front_left_hub_joint
- removed joint base_front_right_axle_joint
- removed joint base_front_right_hub_joint
- removed joint base_to_pantbl
- removed joint p3at_back_left_axle_joint
- removed joint p3at_back_left_hub_joint
- removed joint p3at_back_left_wheel_joint
- removed joint p3at_back_right_axle_joint
- removed joint p3at_back_right_hub_joint
- removed joint p3at_back_right_wheel_joint
- removed joint p3at_front_left_wheel_joint
- removed joint p3at_front_right_wheel_joint
- removed joint pantbl_to_cam
- joint camera_joint: axis 0 1 0 -> (none); limit lower=-1.5 upper=1.5 effort=1000.0 velocity=0.5 -> (none); origin xyz=.15 0 .33 rpy=0 0 0 -> xyz=0.15 0 0.33 rpy=0 0 0
- joint hokuyo_joint: axis 0 1 0 -> (none); origin xyz=.15 0 .3 rpy=0 0 0 -> xyz=0.15 0 0.30 rpy=0 0 0
